Commit message: Auto commit. Files updated at Wed Jan 24 07:41:59 AM +07 2024

File: Module6/ex05/robot_lidar/robotl_description/urdf/depth.urdf.xacro (robot description, xacro)
@@ -14,5 +14,5 @@
             <origin xyz="0.00465 -0.0475 0" rpy="${M_PI/2} 0 ${M_PI/2}"/>
             <geometry>
-                <mesh filename="file://$(find robot_description)/urdf/d455.stl" scale="0.001 0.001 0.001"/>
+                <mesh filename="file://$(find robotl_description)/urdf/d455.stl" scale="0.001 0.001 0.001"/>
                 <!--box size="0.026 0.124 0.029"/-->
             </geometry>
